File: Analog_Teil.sch (EAGLE design)
At the start: 0 parts

Commit message: Filterstufe ohne Schutzeinrichtungen und ohne Spannungsversorgung
Parts:
- added C1, C10, C2, C3, C4: 470n, rcl:C-EUC0805
- added C5, C7, C9: 4.7n, rcl:C-EUC0805
- added C6, C8: 10n, rcl:C-EUC0805
- added IC1, IC3, IC4, IC5, IC6, IC7: OPA388, OPA388:OPA388
- added IC2: INA828ID, INA828ID:INA828ID
- added R1: 50k, rcl:R-EU_R0805
- added R10, R11: 138k, rcl:R-EU_R0805
- added R12, R15: 6.8k, rcl:R-EU_R0805
- added R13, R14, R3, R5: 100k, rcl:R-EU_R0805
- added R2, R4: 48k, rcl:R-EU_R0805
- added R6, R7, R8, R9: 47k, rcl:R-EU_R0805
Connections:
- new net AGND: C5.1, C7.1, R3.1, R5.1
- new net GND1: IC2.REF
- new net N$1: IC2.RG@1, R1.1
- new net N$10: IC3.IN-, IC3.OUT, R4.2, R6.1
- new net N$11: C5.2, IC4.IN+, R7.2
- new net N$12: C8.1, R8.2, R9.1
- new net N$13: C6.2, IC4.IN-, IC4.OUT, R8.1
- new net N$14: C7.2, IC5.IN+, R9.2
- new net N$15: C10.1, C8.2, IC5.IN-, IC5.OUT, R11.1, R14.1
- new net N$17: C10.2, IC6.IN+, R10.2, R11.2, R12.2
- new net N$18: C9.1, IC7.OUT, R12.1
- new net N$19: C9.2, IC6.IN-, R15.1
- new net N$2: IC2.RG@2, R1.2
- new net N$20: IC7.IN-, R15.2
- new net N$21: IC6.OUT, R13.2
- new net N$22: IC7.IN+, R13.1, R14.2
- new net N$3: C1.2, C2.1, R2.1
- new net N$4: C2.2, IC1.IN+, R3.2
- new net N$5: C1.1, IC2.OUT
- new net N$6: C3.1, IC1.IN-, IC1.OUT, R2.2
- new net N$7: C3.2, C4.1, R4.1
- new net N$8: C4.2, IC3.IN+, R5.2
- new net N$9: C6.1, R6.2, R7.1
