File: Analog_Teil.brd (EAGLE design)
At the start: 160 x 100 mm, 53 parts, among them IC1 OPA388, IC2 INA828ID, IC3 OPA388, IC4 OPA388, IC5 OPA388, IC6 OPA388, IC7 OPA388

Commit message: Nächste Erweiterung
Parts:
- added C25, C26, C27, C28, C29, C30: 10p, rcl:C0805
- added JP10, JP11, JP7, JP8, JP9: (no value), jumper:JP3Q
- added JP5, JP6: (no value), jumper:JP2Q
- added R16: 50k, pot:SM-42/43W
Connections:
- removed net N$13: C6.2, IC4.2, IC4.6, R8.1
- new net N$16: JP5.4, R1.1
- new net N$40: JP5.2, R16.1
- new net N$41: JP7.1, JP7.6, R18.1
- new net N$42: C1.1, JP10.5, JP11.5, JP8.5
- new net N$43: JP11.1
- new net N$44: JP9.5
- new net N$45: JP11.3, JP8.3, JP9.3, R6.1
- new net N$46: JP10.3
- new net N$47: C30.2
- new net N$49: C10.1, JP10.1, JP8.1, JP9.1, R11.1, R14.1
- new net N$53: C28.1, C28.2, C6.2, IC4.2, IC4.6, R8.1
- net GND1: now also JP7.3, JP7.5
- net N$1: now also JP5.1, JP5.3; no longer R1.1
- net N$10: now also C29.1, C29.2, JP9.2, JP9.4, JP9.6; no longer R6.1
- net N$15: now also C27.1, C27.2, JP10.2, JP10.4, JP10.6; no longer C10.1, R11.1, R14.1
- net N$18: now also C25.2
- net N$19: now also C26.2
- net N$2: now also R16.2
- net N$20: now also C25.1
- net N$21: now also C26.1, JP11.2, JP11.4, JP11.6
- net N$25: now also JP7.2, JP7.4; no longer R18.1
- net N$5: now also JP8.2, JP8.4, JP8.6; no longer C1.1
- net N$6: now also C30.1

Commit message: Nächste Bearbeitung
Parts:
- removed C11, C12, C13, C14, C15, C16, C17, C18, C19, C20, C21, C22, C23, C24: 100n, rcl:C0805
- removed JP1: (no value), jumper:JP3Q
- removed JP6: (no value), jumper:JP2Q
- added C+1.5, C+3, C+9, C-1.5, C_-9: 100u, ECA-1HM101:CAPPRD350W60D800H1150B
- added C_1+, C_1-, C_H11+, C_H11-, C_H12+, C_H12-, C_N11+, C_N11-, C_N12+, C_N12-, C_T11+, C_T11-, C_T12+, C_T12-: 100n, rcl:C0805
- added TP2, TP3, TP4, TP5, TP6, TP7: TPPAD1-13, testpad:P1-13
- added X1, X2: (no value), con-wago:233-108
- R1, R16: value 50k -> 200
- R_RS+, R_RS-: value 500k -> 1Meg
- renumbered C1 to C_H11.1, C10 to C_N1.1, C2 to C_H11.2, C25 to C_N12.0, C26 to C_N11.0, C27 to C_T12.0, C28 to C_T11.0, C29 to C_H12.0, C3 to C_H12.1, C30 to C_H11.0, C4 to C_H12.2, C5 to C_T11.2, C6 to C_T11.1, C7 to C_T12.2, C8 to C_T12.1, C9 to C_N1.2, IC1 to H11, IC2 to INA_1, IC3 to H12, IC4 to T11, IC5 to T12, IC6 to N11, IC7 to N12, R10 to R_N1.2, R11 to R_N1.1, R12 to R_N1.3, R13 to R_N1.5, R14 to R_N1.6, R15 to R_N1.4, R18 to R_RS+, R19 to R_RS-, R2 to R_H11.1, R3 to R_H11.2, R4 to R_H12.1, R5 to R_H12.2, R6 to R_T11.1, R7 to R_T11.2, R8 to R_T12.1, R9 to R_T12.2
Connections:
- removed net GND1: C11.2, C12.1, C13.2, C14.1, C15.2, C16.1, C17.2, C18.1, C19.2, C20.1, C21.2, C22.1, C23.2, C24.1, INA_1.5, JP7.3, JP7.5
- removed net N$10: C_H12.0.1, C_H12.0.2, H12.2, H12.6, JP9.2, JP9.4, JP9.6, R_H12.1.2
- removed net N$15: C_T12.0.1, C_T12.0.2, C_T12.1.2, JP10.2, JP10.4, JP10.6, T12.2, T12.6
- removed net N$21: C_N11.0.1, JP11.2, JP11.4, JP11.6, N11.6, R_N1.5.2
- removed net N$23: INA_1.2, R_RS-.2
- removed net N$24: INA_1.3, R_RS+.2
- removed net N$26: C11.1, INA_1.4
- removed net N$27: C12.2, INA_1.7
- removed net N$28: C14.2, H11.4
- removed net N$29: C13.1, H11.7
- removed net N$30: C16.2, H12.4
- removed net N$31: C15.1, H12.7
- removed net N$32: C18.2, T11.4
- removed net N$33: C17.1, T11.7
- removed net N$34: C20.2, T12.4
- removed net N$35: C19.1, T12.7
- removed net N$36: C22.2, N11.4
- removed net N$37: C21.1, N11.7
- removed net N$38: C24.2, N12.4
- removed net N$39: C23.1, N12.7
- removed net N$43: JP11.1
- removed net N$44: JP9.5
- removed net N$46: JP10.3
- removed net N$5: INA_1.6, JP8.2, JP8.4, JP8.6
- removed net N$6: C_H11.0.1, C_H12.1.1, H11.2, H11.6, R_H11.1.2
- new net +1.5V: C+1.5.+, C_H11+.1, C_H12+.1, C_N11+.1, C_N12+.1, C_T11+.1, C_T12+.1, H11.7, H12.7, N11.7, N12.7, T11.7, T12.7, X1.B6
- new net +3V: C+3.+, X1.B7
- new net +9V: C+9.+, C_1+.1, INA_1.7, X1.B3
- new net -1.5V: C-1.5.-, C_H11-.2, C_H12-.2, C_N11-.2, C_N12-.2, C_T11-.2, C_T12-.2, H11.4, H12.4, N11.4, N12.4, T11.4, T12.4, X1.B4
- new net -9V: C_-9.-, C_1-.1, INA_1.4, X1.B1
- new net H1_ADC: JP9.5, TP5.TP
- new net H1_OUT: C_H12.0.1, C_H12.0.2, H12.2, H12.6, JP9.2, JP9.4, JP9.6, R_H12.1.2, TP2.TP
- new net INA1_OUT: INA_1.6, JP8.2, JP8.4, JP8.6, TP1.TP
- new net LS+: X2.B4
- new net LS-: X2.B5
- new net N$54: X2.B6
- new net N$55: X1.B8
- new net N$56: X2.B7
- new net N$57: X2.B8
- new net N1_ADC: JP11.1, TP7.TP
- new net N1_OUT: C_N11.0.1, JP11.2, JP11.4, JP11.6, N11.6, R_N1.5.2, TP4.TP
- new net REF: INA_1.5, X2.B3
- new net RS+: INA_1.3, R_RS+.2, X2.B1
- new net RS-: INA_1.2, R_RS-.2, X2.B2
- new net T1_ADC: JP10.3, TP6.TP
- new net T1_OUT: C_T12.0.1, C_T12.0.2, C_T12.1.2, JP10.2, JP10.4, JP10.6, T12.2, T12.6, TP3.TP
- net AGND: now also C+1.5.-, C+3.-, C+9.-, C-1.5.+, C_-9.+, C_1+.2, C_1-.2, C_H11+.2, C_H11-.1, C_H12+.2, C_H12-.1, C_N11+.2, C_N11-.1, C_N12+.2, C_N12-.1, C_T11+.2, C_T11-.1, C_T12+.2, C_T12-.1, JP7.3, JP7.5, R_N1.2.1, X1.B2, X1.B5
- net N$47: now also C_H11.0.1, C_H12.1.1, H11.2, H11.6, R_H11.1.2

Commit message: Überspannungsschutz hinzugefügt
Parts:
- removed JP2: (no value), jumper:JP1
- removed JP3: (no value), jumper:JP2
- removed JP4: (no value), jumper:JP2Q
- added D1, D2: CDZV2_2B, cdzv2_2b:SODFL1006X40N
- added RZ_1: 2k, rcl:R0805
- renumbered TP5 to TP5_H1, TP6 to TP6_T1, TP7 to TP7_N1
Connections:
- removed net H1_ADC: JP9.5, TP5_H1.TP
- removed net N1_ADC: JP11.1, TP7_N1.TP
- removed net T1_ADC: JP10.3, TP6_T1.TP
- new net N$5: D1.1, RZ_1.1
- new net N$6: D1.2, D2.2
- new net TO_ADC1: JP10.3, JP11.1, JP9.5, TP5_H1.TP, TP6_T1.TP, TP7_N1.TP
- net AGND: now also D2.1
- net INA1_OUT: now also RZ_1.2
Changed lines of the file:
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@@
 <layer number="97" name="Info" color="7" fill="1" visible="no" active="no"/>
 <layer number="98" name="Guide" color="6" fill="1" visible="no" active="no"/>
+<layer number="99" name="SpiceOrder" color="5" fill="1" visible="no" active="no"/>
 </layers>
 <board>
@@
 <attribute name="VALUE" x="-49.53" y="-292.1" size="0.0254" layer="27"/>
 </element>
-<element name="JP2" library="jumper" library_urn="urn:adsk.eagle:library:252" package="JP1" package3d_urn="urn:adsk.eagle:package:15455/1" value="" x="-55.88" y="-289.56" smashed="yes">
-<attribute name="NAME" x="-57.531" y="-292.1" size="1.27" layer="25" ratio="10" rot="R90"/>
-<attribute name="VALUE" x="-52.959" y="-292.1" size="1.27" layer="27" ratio="10" rot="R90"/>
-</element>
-<element name="JP3" library="jumper" library_urn="urn:adsk.eagle:library:252" package="JP2" package3d_urn="urn:adsk.eagle:package:15452/1" value="" x="-63.5" y="-288.29" smashed="yes">
-<attribute name="NAME" x="-67.056" y="-286.639" size="1.27" layer="25" ratio="10"/>
-<attribute name="VALUE" x="-67.056" y="-292.608" size="1.27" layer="27" ratio="10"/>
-</element>
-<element name="JP4" library="jumper" library_urn="urn:adsk.eagle:library:252" package="JP2Q" package3d_urn="urn:adsk.eagle:package:15450/1" value="" x="-73.66" y="-288.29" smashed="yes">
-<attribute name="NAME" x="-76.2" y="-285.242" size="1.27" layer="25" ratio="10"/>
-<attribute name="VALUE" x="-69.215" y="-290.83" size="1.27" layer="27" ratio="10" rot="R90"/>
-</element>
 <element name="R16" library="pot" library_urn="urn:adsk.eagle:library:331" package="SM-42/43W" package3d_urn="urn:adsk.eagle:package:22721/1" value="200" x="-82.55" y="-288.29" smashed="yes">
 <attribute name="NAME" x="-84.95" y="-291.915" size="1.27" layer="25"/>
@@
 <attribute name="VALUE" x="-205.74" y="-509.27" size="0.0254" layer="27"/>
 </element>
-<element name="TP5" library="testpad" library_urn="urn:adsk.eagle:library:385" package="P1-13" package3d_urn="urn:adsk.eagle:package:27946/1" value="TPPAD1-13" x="-205.74" y="-514.35" smashed="yes">
+<element name="TP5_H1" library="testpad" library_urn="urn:adsk.eagle:library:385" package="P1-13" package3d_urn="urn:adsk.eagle:package:27946/1" value="TPPAD1-13" x="-205.74" y="-514.35" smashed="yes">
 <attribute name="NAME" x="-206.756" y="-513.08" size="1.27" layer="25" ratio="10"/>
 <attribute name="TP_SIGNAL_NAME" value="" x="-205.74" y="-514.35" size="1.778" layer="27" display="off"/>
 <attribute name="VALUE" x="-205.74" y="-514.35" size="0.0254" layer="27"/>
 </element>
-<element name="TP6" library="testpad" library_urn="urn:adsk.eagle:library:385" package="P1-13" package3d_urn="urn:adsk.eagle:package:27946/1" value="TPPAD1-13" x="-205.74" y="-519.43" smashed="yes">
+<element name="TP6_T1" library="testpad" library_urn="urn:adsk.eagle:library:385" package="P1-13" package3d_urn="urn:adsk.eagle:package:27946/1" value="TPPAD1-13" x="-205.74" y="-519.43" smashed="yes">
 <attribute name="NAME" x="-206.756" y="-518.16" size="1.27" layer="25" ratio="10"/>
 <attribute name="TP_SIGNAL_NAME" value="" x="-205.74" y="-519.43" size="1.778" layer="27" display="off"/>
 <attribute name="VALUE" x="-205.74" y="-519.43" size="0.0254" layer="27"/>
 </element>
-<element name="TP7" library="testpad" library_urn="urn:adsk.eagle:library:385" package="P1-13" package3d_urn="urn:adsk.eagle:package:27946/1" value="TPPAD1-13" x="-205.74" y="-524.51" smashed="yes">
+<element name="TP7_N1" library="testpad" library_urn="urn:adsk.eagle:library:385" package="P1-13" package3d_urn="urn:adsk.eagle:package:27946/1" value="TPPAD1-13" x="-205.74" y="-524.51" smashed="yes">
 <attribute name="NAME" x="-206.756" y="-523.24" size="1.27" layer="25" ratio="10"/>
 <attribute name="TP_SIGNAL_NAME" value="" x="-205.74" y="-524.51" size="1.778" layer="27" display="off"/>
 <attribute name="VALUE" x="-205.74" y="-524.51" size="0.0254" layer="27"/>
+</element>
+<element name="D2" library="cdzv2_2b" package="SODFL1006X40N" value="CDZV2_2B" x="-205.74" y="-534.67" smashed="yes">
+<attribute name="NAME" x="-206.891109375" y="-534.01136875" size="0.8128" layer="25"/>
+<attribute name="VALUE" x="-206.99603125" y="-536.14523125" size="0.8128" layer="27"/>
+</element>
+<element name="D1" library="cdzv2_2b" package="SODFL1006X40N" value="CDZV2_2B" x="-205.74" y="-539.75" smashed="yes">
+<attribute name="NAME" x="-206.891109375" y="-539.09136875" size="0.8128" layer="25"/>
+<attribute name="VALUE" x="-206.99603125" y="-541.22523125" size="0.8128" layer="27"/>
+</element>
+<element name="RZ_1" library="rcl" library_urn="urn:adsk.eagle:library:334" package="R0805" package3d_urn="urn:adsk.eagle:package:23553/2" value="2k" x="-205.74" y="-546.1" smashed="yes">
+<attribute name="NAME" x="-206.375" y="-544.83" size="1.27" layer="25"/>
+<attribute name="SPICEPREFIX" value="R" x="-205.74" y="-546.1" size="1.778" layer="27" display="off"/>
+<attribute name="VALUE" x="-206.375" y="-548.64" size="1.27" layer="27"/>
 </element>
 </elements>
@@
 <contactref element="JP7" pad="5"/>
 <contactref element="R_N1.2" pad="1"/>
+<contactref element="D2" pad="1"/>
+<wire x1="-206.69" y1="-492.76" x2="-206.24" y2="-534.67" width="0" layer="19" extent="1-1"/>
 <wire x1="-204.79" y1="-486.41" x2="-206.69" y2="-492.76" width="0" layer="19" extent="1-1"/>
 <wire x1="-206.69" y1="-480.06" x2="-204.79" y2="-486.41" width="0" layer="19" extent="1-1"/>
@@
 </signal>
 <signal name="INA1_OUT">
-<contactref element="INA_1" pad="6"/>
 <contactref element="JP8" pad="6"/>
 <contactref element="JP8" pad="4"/>
 <contactref element="JP8" pad="2"/>
 <contactref element="TP1" pad="TP"/>
+<contactref element="INA_1" pad="6"/>
+<contactref element="RZ_1" pad="2"/>
+<wire x1="-119.38" y1="-284.48" x2="-204.79" y2="-546.1" width="0" layer="19" extent="1-1"/>
 <wire x1="-116.84" y1="-284.48" x2="-119.38" y2="-284.48" width="0" layer="19" extent="1-1"/>
 <wire x1="-114.3" y1="-284.48" x2="-116.84" y2="-284.48" width="0" layer="19" extent="1-1"/>
@@
 <wire x1="-10.225" y1="-62.865" x2="-13.02" y2="-77.47" width="0" layer="19" extent="1-1"/>
 <wire x1="-15.175" y1="-61.595" x2="-10.225" y2="-62.865" width="0" layer="19" extent="1-1"/>
-</signal>
-<signal name="H1_ADC">
-<contactref element="JP9" pad="5"/>
-<contactref element="TP5" pad="TP"/>
-<wire x1="-123.19" y1="-287.02" x2="-205.74" y2="-514.35" width="0" layer="19" extent="1-1"/>
-</signal>
-<signal name="T1_ADC">
-<contactref element="JP10" pad="3"/>
-<contactref element="TP6" pad="TP"/>
-<wire x1="-134.62" y1="-287.02" x2="-205.74" y2="-519.43" width="0" layer="19" extent="1-1"/>
-</signal>
-<signal name="N1_ADC">
-<contactref element="JP11" pad="1"/>
-<contactref element="TP7" pad="TP"/>
-<wire x1="-146.05" y1="-287.02" x2="-205.74" y2="-524.51" width="0" layer="19" extent="1-1"/>
 </signal>
 <signal name="N$49">
@@
 <contactref element="X2" pad="B8"/>
 </signal>
+<signal name="N$5">
+<contactref element="RZ_1" pad="1"/>
+<contactref element="D1" pad="1"/>
+<wire x1="-206.24" y1="-539.75" x2="-206.69" y2="-546.1" width="0" layer="19" extent="1-1"/>
+</signal>
+<signal name="N$6">
+<contactref element="D1" pad="2"/>
+<contactref element="D2" pad="2"/>
+<wire x1="-205.24" y1="-534.67" x2="-205.24" y2="-539.75" width="0" layer="19" extent="1-1"/>
+</signal>
+<signal name="TO_ADC1">
+<contactref element="JP10" pad="3"/>
+<contactref element="TP6_T1" pad="TP"/>
+<contactref element="JP9" pad="5"/>
+<contactref element="TP5_H1" pad="TP"/>
+<contactref element="JP11" pad="1"/>
+<contactref element="TP7_N1" pad="TP"/>
+<wire x1="-205.74" y1="-519.43" x2="-205.74" y2="-524.51" width="0" layer="19" extent="1-1"/>
+<wire x1="-205.74" y1="-514.35" x2="-205.74" y2="-519.43" width="0" layer="19" extent="1-1"/>
+<wire x1="-146.05" y1="-287.02" x2="-205.74" y2="-514.35" width="0" layer="19" extent="1-1"/>
+<wire x1="-134.62" y1="-287.02" x2="-146.05" y2="-287.02" width="0" layer="19" extent="1-1"/>
+<wire x1="-123.19" y1="-287.02" x2="-134.62" y2="-287.02" width="0" layer="19" extent="1-1"/>
+</signal>
 </signals>
