File: Analog_Teil.brd (EAGLE design)
At the start: 160 x 100 mm, 148 parts, among them J1 35RASMT2BHNTRX, J2 35RASMT2BHNTRX, T11 OPA388, T12 OPA388, T21 OPA388, T22 OPA388

Commit message: Testpunkte, Widerstand hinter Poti, zusätzlich noch Power Supply Platine
Parts:
- added R_INA1_MIN, R_INA2_MIN: 50, rcl:R0805
- added TP15, TP16, TP17, TP18: TPPAD1-13, testpad:P1-13
- R_INA2_VAR: value R_INA2_VAR -> 200
- renumbered R3 to R_INA2_VAR
Connections:
- net N$1 renamed RG1+
- net N$38 renamed RG2+
- removed net N$2: INA_1.8, R_INA1_CONST.2, R_INA1_VAR.2
- removed net N$23: INA_2.8, R_INA2_CONST.2, R_INA2_VAR.2
- removed net N$46: C_H21.0.1, C_H22.1.1, H21.6
- removed net N$47: C_H11.0.1, C_H12.1.1, H11.6
- removed net N$48: C_T21.0.1, R_T22.1.1, T21.6
- removed net N$53: C_T11.0.1, R_T12.1.1, T11.6
- new net H11_OUT: C_H11.0.1, C_H12.1.1, H11.6, TP15.TP
- new net H21_OUT: C_H21.0.1, C_H22.1.1, H21.6, TP17.TP
- new net N$1: R_INA2_MIN.1, R_INA2_VAR.2
- new net N$54: R_INA1_MIN.1, R_INA1_VAR.2
- new net RG1-: INA_1.8, R_INA1_CONST.2, R_INA1_MIN.2
- new net RG2-: INA_2.8, R_INA2_CONST.2, R_INA2_MIN.2
- new net T11_OUT: C_T11.0.1, R_T12.1.1, T11.6, TP16.TP
- new net T21_OUT: C_T21.0.1, R_T22.1.1, T21.6, TP18.TP
- net LS+: now also J2.4; no longer J2.1
- net LS-: now also J2.1; no longer J2.4
- net RS+: now also J1.4; no longer J1.1
- net RS-: now also J1.1; no longer J1.4

Commit message: Schönheitsanpassungen
Parts:
- R_LS1, R_RS: value 1Meg -> 10Meg
- renumbered C_INA2+1 to C_INA2+, C_INA2-1 to C_INA2-
Changed lines of the file:
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@@
 <attribute name="VALUE" x="-41.91" y="-173.99" size="1.27" layer="27"/>
 </element>
-<element name="R_RS" library="rcl" library_urn="urn:adsk.eagle:library:334" package="R0805" package3d_urn="urn:adsk.eagle:package:23553/2" value="1Meg" x="-40.64" y="-196.85" smashed="yes">
+<element name="R_RS" library="rcl" library_urn="urn:adsk.eagle:library:334" package="R0805" package3d_urn="urn:adsk.eagle:package:23553/2" value="10Meg" x="-40.64" y="-196.85" smashed="yes">
 <attribute name="NAME" x="-41.275" y="-195.58" size="1.27" layer="25"/>
 <attribute name="SPICEPREFIX" value="R" x="-40.64" y="-196.85" size="1.778" layer="27" display="off"/>
@@
 <attribute name="VALUE" x="-199.39" y="-610.87" size="1.27" layer="27"/>
 </element>
-<element name="R_LS1" library="rcl" library_urn="urn:adsk.eagle:library:334" package="R0805" package3d_urn="urn:adsk.eagle:package:23553/2" value="1Meg" x="-161.29" y="-601.98" smashed="yes">
+<element name="R_LS1" library="rcl" library_urn="urn:adsk.eagle:library:334" package="R0805" package3d_urn="urn:adsk.eagle:package:23553/2" value="10Meg" x="-161.29" y="-601.98" smashed="yes">
 <attribute name="NAME" x="-161.925" y="-600.71" size="1.27" layer="25"/>
 <attribute name="SPICEPREFIX" value="R" x="-259.08" y="-721.36" size="1.778" layer="27" display="off"/>
@@
 <attribute name="VALUE" x="-207.01" y="-655.955" size="1.27" layer="27"/>
 </element>
-<element name="C_INA2-1" library="rcl" library_urn="urn:adsk.eagle:library:334" package="C0805" package3d_urn="urn:adsk.eagle:package:23617/2" value="100n" x="-205.74" y="-664.21" smashed="yes">
+<element name="C_INA2-" library="rcl" library_urn="urn:adsk.eagle:library:334" package="C0805" package3d_urn="urn:adsk.eagle:package:23617/2" value="100n" x="-205.74" y="-664.21" smashed="yes">
 <attribute name="NAME" x="-207.01" y="-662.94" size="1.27" layer="25"/>
 <attribute name="SPICEPREFIX" value="C" x="-205.74" y="-657.86" size="1.778" layer="27" display="off"/>
 <attribute name="VALUE" x="-207.01" y="-666.75" size="1.27" layer="27"/>
 </element>
-<element name="C_INA2+1" library="rcl" library_urn="urn:adsk.eagle:library:334" package="C0805" package3d_urn="urn:adsk.eagle:package:23617/2" value="100n" x="-205.74" y="-657.86" smashed="yes">
+<element name="C_INA2+" library="rcl" library_urn="urn:adsk.eagle:library:334" package="C0805" package3d_urn="urn:adsk.eagle:package:23617/2" value="100n" x="-205.74" y="-657.86" smashed="yes">
 <attribute name="NAME" x="-207.01" y="-656.59" size="1.27" layer="25"/>
 <attribute name="SPICEPREFIX" value="C" x="-205.74" y="-664.21" size="1.778" layer="27" display="off"/>
@@
 <contactref element="JP7" pad="2"/>
 <contactref element="JP7" pad="5"/>
-<contactref element="C_INA2-1" pad="2"/>
-<contactref element="C_INA2+1" pad="2"/>
+<contactref element="C_INA2-" pad="2"/>
+<contactref element="C_INA2+" pad="2"/>
 <contactref element="C_N22+" pad="2"/>
 <contactref element="C_N22-" pad="1"/>
@@
 <contactref element="INA_2" pad="4"/>
 <contactref element="JP7" pad="1"/>
-<contactref element="C_INA2-1" pad="1"/>
+<contactref element="C_INA2-" pad="1"/>
 <wire x1="-205.74" y1="-652.78" x2="-201.295" y2="-559.01" width="0" layer="19" extent="1-1"/>
 <wire x1="-206.69" y1="-664.21" x2="-205.74" y2="-652.78" width="0" layer="19" extent="1-1"/>
@@
 <contactref element="INA_2" pad="7"/>
 <contactref element="JP7" pad="3"/>
-<contactref element="C_INA2+1" pad="1"/>
+<contactref element="C_INA2+" pad="1"/>
 <wire x1="-200.66" y1="-652.78" x2="-203.835" y2="-553.51" width="0" layer="19" extent="1-1"/>
 <wire x1="-206.69" y1="-657.86" x2="-200.66" y2="-652.78" width="0" layer="19" extent="1-1"/>
