File: EMG_digital_Part.brd (EAGLE design)
At the start: 160 x 100 mm, 34 parts

Commit message: Pinout erweitert, Analog u. digital Power Caps, Taster, LEDs
Parts:
- removed JP1: (no value), jumper:JP2W
- added C22, C24, C26, C29, C32, C34, C35: 4.7uF, resistor:C0603
- added C23, C25, C27, C28, C30, C31, C33, C36, C43: 100nF, resistor:C0603
- added C38, C44: 0.47uF, resistor:C0603
- added JP2: (no value), custom_jumper:JP2
- added R36: 10R, _MSP430:R0805
- added SV4: (no value), con-lstb:MA08-1
- RESET: value (none) -> RESET
- moved C101 12.0 mm to (-55.9, -33.0), turned to 90 degrees
- moved C100 8.13 mm to (-47.0, -33.0), turned to 90 degrees
- moved XT1 6.35 mm to (-50.8, -29.2)
- renumbered BTN1 to BTN_3, BTN2 to BTN_2, BTN3 to BTN_4, BTN4 to BTN_1
Connections:
- removed net N$16: SV1.10
- removed net N$7: SV1.9
- new net AUXVCC1: C26.1, C27.1, U$1.22
- new net AUXVCC2: C24.1, C25.1, U$1.21
- new net AUXVCC3: C43.1, C44.1, U$1.29
- new net AVCC: C29.1, C31.1, R36.2, U$1.19
- new net DVSYS: C34.1, C36.1, U$1.23, U$1.75
- new net P1.4: U$1.33
- new net P1.5: U$1.32
- new net P1.6: U$1.40
- new net P1.7: U$1.41
- new net P2.4: U$1.47
- new net P2.5: U$1.48
- new net P2.6: U$1.49
- new net P2.7: U$1.50
- new net P4.1: U$1.60
- new net P4.2: U$1.61
- new net P4.3: U$1.62
- new net P4.4: U$1.63
- new net P4.5: U$1.64
- new net P4.6: U$1.65
- new net P4.7: U$1.66
- new net P5.6: SV1.9, U$1.73
- new net P5.7: SV1.10, U$1.74
- new net P6.0: SV4.1, U$1.77
- new net P6.1: SV4.2, U$1.78
- new net P6.2: SV4.3, U$1.79
- new net P6.3: SV4.4, U$1.80
- new net P6.4: SV4.5, U$1.81
- new net P6.5: SV4.6, U$1.82
- new net P6.6: SV4.7, U$1.83
- new net P6.7: SV4.8, U$1.84
- new net P7.0: SV2.1, U$1.85
- new net P7.1: SV2.2, U$1.86
- new net P7.2: SV2.3, U$1.87
- new net P7.3: SV2.4, U$1.88
- new net P7.4: SV2.5, U$1.89
- new net P7.5: SV2.6, U$1.90
- new net P7.6: SV2.7, U$1.91
- new net P7.7: SV2.8, U$1.92
- new net P8.0: SV2.9, U$1.93
- new net P8.1: SV2.10, U$1.94
- new net VASYS1/2: C22.1, C23.1, C28.1, C32.1, U$1.20, U$1.9
- net AGND: now also C22.2, C23.2, C28.2, C29.2, C30.2, C31.2, C32.2
- net DGND: now also C24.2, C25.2, C26.2, C27.2, C33.2, C34.2, C35.2, C36.2, C38.2, C43.2, C44.2, U$1.38, U$1.39
- net DVCC: now also C33.1, C35.1, JP2.2, R36.1; no longer JP1.2
- net EXT: now also JP2.3; no longer JP1.3
- net INT: now also JP2.1; no longer JP1.1
- net VCORE: now also C38.1
- net VREF: now also C30.1

Commit message: Initial version of analog and digital design
Parts:
- removed R36: 10R, _MSP430:R0805
- removed SV1, SV2: (no value), con-lstb:MA05-2
- removed SV3: (no value), con-lstb:MA05-1
- removed SV4: (no value), con-lstb:MA08-1
- added CLOCK, P1: (no value), con-lstb:MA05-1
- added DGND1, DGND2: (no value), pinhead:1X01
- added P2, P3, P4, P5: (no value), con-lstb:MA08-1
- added P6: (no value), con-lstb:MA06-1
- added R1: 10R, resistor:R0805
- added R2: 0R, resistor:R0805
- C100, C101, C110, C22, C23, C24, C25, C26, C27, C28, C29, C30, C31, C32, C33, C34, C35, C36, C38, C43, C44: device resistor:C0603 -> resistor:C0805
- R101, R110, R111, R112, R114, R115, R116, R117, R120, R121, R122, R123: device resistor:R0603 -> resistor:R0805
- moved BTN_3 283.4 mm to (228.6, 59.7)
- moved U$1 272.6 mm to (232.4, 108.0)
- moved LED2 256.3 mm to (157.5, 83.8)
- moved LED4 256.3 mm to (157.5, 78.7)
- moved LED5 256.3 mm to (167.6, 78.7)
- moved LED6 256.3 mm to (157.5, 73.7)
- moved LED3 248.6 mm to (153.7, 88.9)
- moved R117 229.0 mm to (144.8, 96.5)
- moved R114 228.9 mm to (144.8, 90.2)
- moved JTAG 223.2 mm to (165.1, 137.2), turned to 180 degrees
- moved R115 209.3 mm to (129.5, 71.1)
- moved R116 209.3 mm to (124.5, 71.1)
- moved R110 209.3 mm to (124.5, 64.8)
- moved R111 209.3 mm to (129.5, 64.8)
- moved R112 209.3 mm to (134.6, 64.8)
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Connections:
- removed net P1.4: U$1.33
- removed net P1.5: U$1.32
- removed net P1.6: U$1.40
- removed net P1.7: U$1.41
- removed net P2.4: U$1.47
- removed net P2.5: U$1.48
- removed net P2.6: U$1.49
- removed net P2.7: U$1.50
- removed net P3.0: SV1.1, U$1.51
- removed net P3.1: SV1.2, U$1.52
- removed net P3.2: SV1.3, U$1.53
- removed net P3.3: SV1.4, U$1.54
- removed net P3.4: SV1.5, U$1.55
- removed net P3.5: SV1.6, U$1.56
- removed net P3.6: SV1.7, U$1.57
- removed net P3.7: SV1.8, U$1.58
- removed net P4.4: U$1.63
- removed net P5.6: SV1.9, U$1.73
- removed net P5.7: SV1.10, U$1.74
- removed net P6.1: SV4.2, U$1.78
- removed net P6.6: SV4.7, U$1.83
- removed net P6.7: SV4.8, U$1.84
- removed net P7.0: SV2.1, U$1.85
- removed net P7.1: SV2.2, U$1.86
- removed net P7.2: SV2.3, U$1.87
- removed net P7.3: SV2.4, U$1.88
- removed net P7.4: SV2.5, U$1.89
- removed net P7.5: SV2.6, U$1.90
- removed net P7.6: SV2.7, U$1.91
- removed net P7.7: SV2.8, U$1.92
- removed net P8.0: SV2.9, U$1.93
- removed net P8.1: SV2.10, U$1.94
- new net N$12: P1.1, U$1.41
- new net N$13: P1.2, U$1.40
- new net N$14: P1.3, U$1.34
- new net N$15: P1.4, U$1.36
- new net N$16: P1.5, U$1.37
- new net N$17: P5.2, U$1.68
- new net N$18: P5.3, U$1.69
- new net N$19: P5.4, U$1.70
- new net N$20: P2.8, U$1.42
- new net N$22: P2.7, U$1.43
- new net N$23: P2.6, U$1.44
- new net N$24: P2.5, U$1.45
- new net N$25: P2.4, U$1.47
- new net N$26: P2.3, U$1.48
- new net N$28: P2.2, U$1.49
- new net N$29: P2.1, U$1.50
- new net N$31: P3.8, U$1.51
- new net N$32: P3.7, U$1.52
- new net N$33: P3.6, U$1.53
- new net N$34: P3.5, U$1.54
- new net N$35: P3.4, U$1.55
- new net N$37: P3.3, U$1.56
- new net N$38: P3.2, U$1.57
- new net N$39: P3.1, U$1.58
- new net N$40: P5.5, U$1.71
- new net N$41: P5.6, U$1.72
- new net N$42: P5.7, U$1.73
- new net N$43: P5.8, U$1.74
- new net N$44: P4.5, U$1.63
- new net N$5: P6.2, U$1.78
- new net P4.0: P4.1, U$1.59
- net ACLK: now also CLOCK.3, U$1.35; no longer SV3.3, U$1.44
- net ACT_LED: now also U$1.93; no longer U$1.59
- net AGND: now also R2.2, U$1.10
- net AVCC: now also R1.2; no longer R36.2
- net BTN1: now also U$1.91; no longer U$1.37
- net BTN2: now also U$1.92; no longer U$1.36
- net BTN3: now also U$1.83; no longer BTN_3.2, R122.2, U$1.35
- net BTN4: now also U$1.84; no longer U$1.34
- net DGND: now also CLOCK.1, DGND1.1, DGND2.1, R2.1; no longer SV3.1
- net DVCC: now also R1.1; no longer R36.1
- net LED1: now also U$1.85; no longer U$1.67
- net LED2: now also U$1.86; no longer U$1.68
- net LED3: now also U$1.87; no longer U$1.69
- net LED4: now also U$1.88; no longer U$1.70
- net LED5: now also U$1.89; no longer U$1.71
- net LED6: now also U$1.90; no longer U$1.72
- net MCLK: now also CLOCK.4, U$1.33; no longer SV3.4, U$1.43
- net N$3: now also P5.1, U$1.67; no longer U$1.10
- net P4.1: now also P4.2
- net P4.2: now also P4.3
- net P4.3: now also P4.4
- net P4.5: now also P4.6
- net P4.6: now also P4.7
- net P4.7: now also P4.8
- net P6.0: now also BTN_3.2, P6.1, R122.2; no longer SV4.1
- net P6.2: now also P6.3; no longer SV4.3
- net P6.3: now also P6.4; no longer SV4.4
- net P6.4: now also P6.5; no longer SV4.5
- net P6.5: now also P6.6; no longer SV4.6
- net RTCCLK: now also CLOCK.2, U$1.94; no longer SV3.2, U$1.45
- net SMCLK: now also CLOCK.5, U$1.32; no longer SV3.5, U$1.42
Other:
- board size 160 x 100 mm -> 276.8 x 145.7 mm
