File: EMG_digital_Part.sch (EAGLE design)
At the start: 34 parts

Commit message: ....
Parts:
- removed JP1: (no value), jumper:JP2W
- added C22, C24, C26, C29, C32, C34, C35: 4.7uF, resistor:C-EUC0603
- added C23, C25, C27, C28, C30, C31, C33, C36, C43: 100nF, resistor:C-EUC0603
- added C38, C44: 0.47uF, resistor:C-EUC0603
- added JP2: (no value), custom_jumper:JP2E
- added R36: 10R, _MSP430:RES0805
- RESET: value (none) -> RESET
Connections:
- new net AUXVCC1: C26.1, C27.1
- new net AUXVCC2: C24.1, C25.1
- new net AUXVCC3: C43.1, C44.1
- new net AVCC: C29.1, C31.1, R36.2, U$1.AVCC
- new net DVSYS_VDSYS: C34.1, C36.1
- new net N$5: U$1.AUXVCC1
- new net N$6: U$1.AUXVCC2
- new net N$8: U$1.AUXVCC3
- new net VASYS1/2: C22.1, C23.1, C28.1, C32.1, U$1.VASYS1, U$1.VASYS2
- net AGND: now also C22.2, C23.2, C28.2, C29.2, C30.2, C31.2, C32.2
- net DGND: now also C24.2, C25.2, C26.2, C27.2, C33.2, C34.2, C35.2, C36.2, C38.2, C43.2, C44.2, U$1.COM0, U$1.COM1
- net DVCC: now also C33.1, C35.1, JP2.2, R36.1; no longer JP1.2
- net EXT: now also JP2.3; no longer JP1.3
- net INT: now also JP2.1; no longer JP1.1
- net VCORE: now also C38.1
- net VREF: now also C30.1
Other:
- note added: "Analog Power"
- note added: "Digital Power"
- moved on the sheet: BTN1, BTN2, BTN3, BTN4, C100, C101, C110, JTAG, LED1, LED2, LED3, LED4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

Commit message: Pinout erweitert, Analog u. digital Power Caps, Taster, LEDs
Parts:
- added SV4: (no value), con-lstb:MA08-1
- renumbered BTN1 to BTN_3, BTN2 to BTN_2, BTN3 to BTN_4, BTN4 to BTN_1
Connections:
- removed net DVSYS_VDSYS: C34.1, C36.1
- removed net N$16: SV1.10
- removed net N$5: U$1.AUXVCC1
- removed net N$6: U$1.AUXVCC2
- removed net N$7: SV1.9
- removed net N$8: U$1.AUXVCC3
- new net DVSYS: C34.1, C36.1, U$1.VDSYS1, U$1.VDSYS2
- new net P1.4: U$1.P1.4
- new net P1.5: U$1.P1.5
- new net P1.6: U$1.P1.6
- new net P1.7: U$1.P1.7
- new net P2.4: U$1.P2.4
- new net P2.5: U$1.P2.5
- new net P2.6: U$1.P2.6
- new net P2.7: U$1.P2.7
- new net P4.1: U$1.P4.1
- new net P4.2: U$1.P4.2
- new net P4.3: U$1.P4.3
- new net P4.4: U$1.P4.4
- new net P4.5: U$1.P4.5
- new net P4.6: U$1.P4.6
- new net P4.7: U$1.P4.7
- new net P5.6: SV1.9, U$1.P5.6
- new net P5.7: SV1.10, U$1.P5.7
- new net P6.0: SV4.1, U$1.P6.0
- new net P6.1: SV4.2, U$1.P6.1
- new net P6.2: SV4.3, U$1.P6.2
- new net P6.3: SV4.4, U$1.P6.3
- new net P6.4: SV4.5, U$1.P6.4
- new net P6.5: SV4.6, U$1.P6.5
- new net P6.6: SV4.7, U$1.P6.6
- new net P6.7: SV4.8, U$1.P6.7
- new net P7.0: SV2.1, U$1.P7.0
- new net P7.1: SV2.2, U$1.P7.1
- new net P7.2: SV2.3, U$1.P7.2
- new net P7.3: SV2.4, U$1.P7.3
- new net P7.4: SV2.5, U$1.P7.4
- new net P7.5: SV2.6, U$1.P7.5
- new net P7.6: SV2.7, U$1.P7.6
- new net P7.7: SV2.8, U$1.P7.7
- new net P8.0: SV2.9, U$1.P8.0
- new net P8.1: SV2.10, U$1.P8.1
- net AUXVCC1: now also U$1.AUXVCC1
- net AUXVCC2: now also U$1.AUXVCC2
- net AUXVCC3: now also U$1.AUXVCC3
Other:
- note added: "Pinout #1"
- note added: "Pinout#2"
- note removed: "Pinout"

Commit message: Initial version of analog and digital design
Parts:
- removed R36: 10R, _MSP430:RES0805
- removed SV1, SV2: (no value), con-lstb:MA05-2
- removed SV3: (no value), con-lstb:MA05-1
- removed SV4: (no value), con-lstb:MA08-1
- added CLOCK, P1: (no value), con-lstb:MA05-1
- added DGND1, DGND2: (no value), pinhead:PINHD-1X1
- added P2, P3, P4, P5: (no value), con-lstb:MA08-1
- added P6: (no value), con-lstb:MA06-1
- added R1: 10R, resistor:R-EU_R0805
- added R2: 0R, resistor:R-EU_R0805
- C100, C101, C110, C22, C23, C24, C25, C26, C27, C28, C29, C30, C31, C32, C33, C34, C35, C36, C38, C43, C44: device resistor:C-EUC0603 -> resistor:C-EUC0805
- R101, R110, R111, R112, R114, R115, R116, R117, R120, R121, R122, R123: device resistor:R-EU_R0603 -> resistor:R-EU_R0805
Connections:
- removed net P1.4: U$1.P1.4
- removed net P1.5: U$1.P1.5
- removed net P1.6: U$1.P1.6
- removed net P1.7: U$1.P1.7
- removed net P2.4: U$1.P2.4
- removed net P2.5: U$1.P2.5
- removed net P2.6: U$1.P2.6
- removed net P2.7: U$1.P2.7
- removed net P3.0: SV1.1, U$1.P3.0
- removed net P3.1: SV1.2, U$1.P3.1
- removed net P3.2: SV1.3, U$1.P3.2
- removed net P3.3: SV1.4, U$1.P3.3
- removed net P3.4: SV1.5, U$1.P3.4
- removed net P3.5: SV1.6, U$1.P3.5
- removed net P3.6: SV1.7, U$1.P3.6
- removed net P3.7: SV1.8, U$1.P3.7
- removed net P4.4: U$1.P4.4
- removed net P5.6: SV1.9, U$1.P5.6
- removed net P5.7: SV1.10, U$1.P5.7
- removed net P6.1: SV4.2, U$1.P6.1
- removed net P6.6: SV4.7, U$1.P6.6
- removed net P6.7: SV4.8, U$1.P6.7
- removed net P7.0: SV2.1, U$1.P7.0
- removed net P7.1: SV2.2, U$1.P7.1
- removed net P7.2: SV2.3, U$1.P7.2
- removed net P7.3: SV2.4, U$1.P7.3
- removed net P7.4: SV2.5, U$1.P7.4
- removed net P7.5: SV2.6, U$1.P7.5
- removed net P7.6: SV2.7, U$1.P7.6
- removed net P7.7: SV2.8, U$1.P7.7
- removed net P8.0: SV2.9, U$1.P8.0
- removed net P8.1: SV2.10, U$1.P8.1
- new net N$12: P1.1, U$1.P1.7
- new net N$13: P1.2, U$1.P1.6
- new net N$14: P1.3, U$1.P1.3
- new net N$15: P1.4, U$1.P1.1
- new net N$16: P1.5, U$1.P1.0
- new net N$17: P5.2, U$1.P5.1
- new net N$18: P5.3, U$1.P5.2
- new net N$19: P5.4, U$1.P5.3
- new net N$20: P2.8, U$1.P2.0
- new net N$22: P2.7, U$1.P2.1
- new net N$23: P2.6, U$1.P2.2
- new net N$24: P2.5, U$1.P2.3
- new net N$25: P2.4, U$1.P2.4
- new net N$26: P2.3, U$1.P2.5
- new net N$28: P2.2, U$1.P2.6
- new net N$29: P2.1, U$1.P2.7
- new net N$31: P3.8, U$1.P3.0
- new net N$32: P3.7, U$1.P3.1
- new net N$33: P3.6, U$1.P3.2
- new net N$34: P3.5, U$1.P3.3
- new net N$35: P3.4, U$1.P3.4
- new net N$37: P3.3, U$1.P3.5
- new net N$38: P3.2, U$1.P3.6
- new net N$39: P3.1, U$1.P3.7
- new net N$40: P5.5, U$1.P5.4
- new net N$41: P5.6, U$1.P5.5
- new net N$42: P5.7, U$1.P5.6
- new net N$43: P5.8, U$1.P5.7
- new net N$44: P4.5, U$1.P4.4
- new net N$5: P6.2, U$1.P6.1
- new net P4.0: P4.1, U$1.P4.0
- net ACLK: now also CLOCK.3, U$1.P1.2; no longer SV3.3, U$1.P2.2
- net ACT_LED: now also U$1.P8.0; no longer U$1.P4.0
- net AGND: now also R2.2, U$1.AVSS2
- net AVCC: now also R1.2; no longer R36.2
- net BTN1: now also U$1.P7.6; no longer U$1.P1.0
- net BTN2: now also U$1.P7.7; no longer U$1.P1.1
- net BTN3: now also U$1.P6.6; no longer BTN_3.S, R122.2, U$1.P1.2
- net BTN4: now also U$1.P6.7; no longer U$1.P1.3
- net DGND: now also CLOCK.1, DGND1.1, DGND2.1, R2.1; no longer SV3.1
- net DVCC: now also R1.1; no longer R36.1
- net LED1: now also U$1.P7.0; no longer U$1.P5.0
- net LED2: now also U$1.P7.1; no longer U$1.P5.1
- net LED3: now also U$1.P7.2; no longer U$1.P5.2
- net LED4: now also U$1.P7.3; no longer U$1.P5.3
- net LED5: now also U$1.P7.4; no longer U$1.P5.4
- net LED6: now also U$1.P7.5; no longer U$1.P5.5
- net MCLK: now also CLOCK.4, U$1.P1.4; no longer SV3.4, U$1.P2.1
- net N$3: now also P5.1, U$1.P5.0; no longer U$1.AVSS2
- net P4.1: now also P4.2
- net P4.2: now also P4.3
- net P4.3: now also P4.4
- net P4.5: now also P4.6
- net P4.6: now also P4.7
- net P4.7: now also P4.8
- net P6.0: now also BTN_3.S, P6.1, R122.2; no longer SV4.1
- net P6.2: now also P6.3; no longer SV4.3
- net P6.3: now also P6.4; no longer SV4.4
- net P6.4: now also P6.5; no longer SV4.5
- net P6.5: now also P6.6; no longer SV4.6
- net RTCCLK: now also CLOCK.2, U$1.P8.1; no longer SV3.2, U$1.P2.3
- net SMCLK: now also CLOCK.5, U$1.P1.5; no longer SV3.5, U$1.P2.0
Other:
- note added: "AGND <--> DGND"
- note added: "Channel 1"
- note added: "Channel 2"
- note added: "GND Pins"
- note added: "Input SigmaDelta"
- note added: "Pinout"
- note removed: "Pinout #1"
- note removed: "Pinout#2"
- moved on the sheet: C22, C23, C28, C29, C30, C31, C32, LED1, LED2, LED3, LED4, LED5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
