File: EMG_SS19_Version_1.0.sch (EAGLE design)
At the start: 212 parts, among them T11 OPA388, T12 OPA388, T21 OPA388, T22 OPA388

Commit message: next version of digital part implementation
Connections:
- removed net P6.0: BTN_3.S, P6.1, R122.2, U$1.P6.0
- new net N$93: P6.1, U$1.P6.0
- new net N$95: U$1.P8.0
- net ACT_LED: now also U$1.P6.6; no longer U$1.P8.0
- net BTN1: now also U$1.P7.1; no longer U$1.P7.6
- net BTN2: now also U$1.P7.0; no longer U$1.P7.7
- net BTN3: now also BTN_3.S, R122.2; no longer U$1.P6.6
- net LED1: now also U$1.P7.7; no longer U$1.P7.0
- net LED2: now also U$1.P7.6; no longer U$1.P7.1
Changed lines of the file:
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@@
 </segment>
 <segment>
-<pinref part="U$1" gate="G$1" pin="P7.6"/>
-<wire x1="109.22" y1="113.03" x2="114.3" y2="113.03" width="0.1524" layer="91"/>
-<wire x1="114.3" y1="113.03" x2="114.3" y2="114.3" width="0.1524" layer="91"/>
-<label x="114.3" y="114.3" size="1.778" layer="95"/>
+<pinref part="U$1" gate="G$1" pin="P7.1"/>
+<wire x1="109.22" y1="125.73" x2="114.3" y2="125.73" width="0.1524" layer="91"/>
+<wire x1="114.3" y1="125.73" x2="114.3" y2="127" width="0.1524" layer="91"/>
+<label x="114.3" y="127" size="1.778" layer="95"/>
 </segment>
 </net>
@@
 </segment>
 <segment>
-<pinref part="U$1" gate="G$1" pin="P7.7"/>
-<wire x1="109.22" y1="110.49" x2="114.3" y2="110.49" width="0.1524" layer="91"/>
-<wire x1="114.3" y1="110.49" x2="114.3" y2="111.76" width="0.1524" layer="91"/>
-<label x="114.3" y="111.76" size="1.778" layer="95"/>
-</segment>
-</net>
-<net name="P6.0" class="0">
-<segment>
-<wire x1="332.74" y1="157.48" x2="332.74" y2="154.94" width="0.1524" layer="91"/>
-<wire x1="332.74" y1="154.94" x2="332.74" y2="152.4" width="0.1524" layer="91"/>
-<wire x1="332.74" y1="154.94" x2="340.36" y2="154.94" width="0.1524" layer="91"/>
-<junction x="332.74" y="154.94"/>
-<label x="340.36" y="154.94" size="1.778" layer="95"/>
-<pinref part="R122" gate="G$1" pin="2"/>
-<pinref part="BTN_3" gate="G$1" pin="S"/>
-</segment>
-<segment>
-<pinref part="U$1" gate="G$1" pin="P6.0"/>
-<wire x1="109.22" y1="154.94" x2="132.08" y2="154.94" width="0.1524" layer="91"/>
-<pinref part="P6" gate="1" pin="1"/>
+<pinref part="U$1" gate="G$1" pin="P7.0"/>
+<wire x1="109.22" y1="128.27" x2="114.3" y2="128.27" width="0.1524" layer="91"/>
+<wire x1="114.3" y1="128.27" x2="114.3" y2="129.54" width="0.1524" layer="91"/>
+<label x="114.3" y="129.54" size="1.778" layer="95"/>
 </segment>
 </net>
@@
 </segment>
 <segment>
-<pinref part="U$1" gate="G$1" pin="P7.0"/>
-<wire x1="109.22" y1="128.27" x2="114.3" y2="128.27" width="0.1524" layer="91"/>
-<wire x1="114.3" y1="128.27" x2="114.3" y2="129.54" width="0.1524" layer="91"/>
-<label x="114.3" y="129.54" size="1.778" layer="95"/>
+<pinref part="U$1" gate="G$1" pin="P7.7"/>
+<wire x1="109.22" y1="110.49" x2="114.3" y2="110.49" width="0.1524" layer="91"/>
+<wire x1="114.3" y1="110.49" x2="114.3" y2="111.76" width="0.1524" layer="91"/>
+<label x="114.3" y="111.76" size="1.778" layer="95"/>
 </segment>
 </net>
@@
 </segment>
 <segment>
-<pinref part="U$1" gate="G$1" pin="P7.1"/>
-<wire x1="109.22" y1="125.73" x2="114.3" y2="125.73" width="0.1524" layer="91"/>
-<wire x1="114.3" y1="125.73" x2="114.3" y2="127" width="0.1524" layer="91"/>
-<label x="114.3" y="127" size="1.778" layer="95"/>
+<pinref part="U$1" gate="G$1" pin="P7.6"/>
+<wire x1="109.22" y1="113.03" x2="114.3" y2="113.03" width="0.1524" layer="91"/>
+<wire x1="114.3" y1="113.03" x2="114.3" y2="114.3" width="0.1524" layer="91"/>
+<label x="114.3" y="114.3" size="1.778" layer="95"/>
 </segment>
 </net>
@@
 </segment>
 <segment>
-<pinref part="U$1" gate="G$1" pin="P8.0"/>
-<wire x1="109.22" y1="101.6" x2="114.3" y2="101.6" width="0.1524" layer="91"/>
-<label x="114.3" y="101.6" size="1.778" layer="95"/>
+<pinref part="U$1" gate="G$1" pin="P6.6"/>
+<wire x1="109.22" y1="139.7" x2="114.3" y2="139.7" width="0.1524" layer="91"/>
+<label x="114.3" y="139.7" size="1.778" layer="95"/>
 </segment>
 </net>
@@
 <net name="BTN3" class="0">
 <segment>
-<pinref part="U$1" gate="G$1" pin="P6.6"/>
-<wire x1="109.22" y1="139.7" x2="114.3" y2="139.7" width="0.1524" layer="91"/>
-<label x="114.3" y="139.7" size="1.778" layer="95"/>
+<wire x1="332.74" y1="157.48" x2="332.74" y2="154.94" width="0.1524" layer="91"/>
+<wire x1="332.74" y1="154.94" x2="332.74" y2="152.4" width="0.1524" layer="91"/>
+<wire x1="332.74" y1="154.94" x2="340.36" y2="154.94" width="0.1524" layer="91"/>
+<junction x="332.74" y="154.94"/>
+<pinref part="R122" gate="G$1" pin="2"/>
+<pinref part="BTN_3" gate="G$1" pin="S"/>
+<label x="340.36" y="154.94" size="1.778" layer="95"/>
 </segment>
 </net>
@@
 </segment>
 </net>
+<net name="N$93" class="0">
+<segment>
+<pinref part="U$1" gate="G$1" pin="P6.0"/>
+<pinref part="P6" gate="1" pin="1"/>
+<wire x1="109.22" y1="154.94" x2="132.08" y2="154.94" width="0.1524" layer="91"/>
+</segment>
+</net>
+<net name="N$95" class="0">
+<segment>
+<pinref part="U$1" gate="G$1" pin="P8.0"/>
+<wire x1="109.22" y1="101.6" x2="114.3" y2="101.6" width="0.1524" layer="91"/>
+</segment>
+</net>

Commit message: first version of analog & digital part completed --> ready for review
Connections:
- removed net +3V: C+3.+, JP7.8
- removed net N$95: U$1.P8.0
- net ACT_LED: now also U$1.P7.2; no longer U$1.P6.6
- net AGND: now also U$1.SD2N0; no longer U$1.SD4N0
- net BTN3: now also U$1.P6.6
- net DGND: now also U$1.SD4N0, U$1.SD4P0; no longer U$1.SD2N0, U$1.SD2P0
- net DVCC: now also C+3.+, JP7.8
- net LED1: now also U$1.P8.0; no longer U$1.P7.7
- net LED3: now also U$1.P7.3; no longer U$1.P7.2
- net LED4: now also U$1.P7.4; no longer U$1.P7.3
- net LED5: now also U$1.P7.5; no longer U$1.P7.4
- net LED6: now also U$1.P7.7; no longer U$1.P7.5
- net SD_IN_2P: now also U$1.SD2P0; no longer U$1.SD4P0
