File: EMG_SS19_Version_2.0.sch (EAGLE design)
At the start: 219 parts, among them T11 OPA388, T12 OPA388, T21 OPA388, T22 OPA388

Commit message: buttons replaced, addad some labeling
Parts:
- removed BTN_1, BTN_2, BTN_3, BTN_4, RESET_BTN: PUSH-BUTTONSURFACE-MOUNT, Taster:PUSH-BUTTONSURFACE-MOUNT
- added SW1, SW2, SW3, SW4, SW5: B3S-1000, B3S-1000:B3S-1000
Connections:
- new net N$56: SW2.1
- net BTN1: now also SW1.1; no longer BTN_1.OUT1, BTN_1.OUT2
- net BTN2: now also SW2.3; no longer BTN_2.OUT1, BTN_2.OUT2
- net BTN3: now also SW3.1; no longer BTN_3.OUT1, BTN_3.OUT2
- net BTN4: now also SW4.3; no longer BTN_4.OUT1, BTN_4.OUT2
- net DGND: now also SW1.4, SW2.4, SW3.4, SW4.4, SW5.4; no longer BTN_1.IN1, BTN_1.IN2, BTN_2.IN1, BTN_2.IN2, BTN_3.IN1, BTN_3.IN2, BTN_4.IN1, BTN_4.IN2, RESET_BTN.OUT1, RESET_BTN.OUT2
- net RESET: now also SW5.3; no longer RESET_BTN.IN1, RESET_BTN.IN2
